File: USB OverDrive.kicad_sch (KiCad schematic)
At the start: 91 parts, among them J1 USB3_A, J2 USB3_A, J3 USB3_A, J4 USB3_A, P1 USB_C_Plug, U1 TUSB8041, U2 1.1V, U3 5.0V, U4 3.3V, U5 TPS2561, U6 TPS2561, Y1 24MHZ

Commit message: sadlkfjsadlkf
Parts:
- added C16, C17: 0.1uF, Capacitor_SMD:C_0201_0603Metric, symbol Device:C
- added C20, C21: 150uF, Capacitor_SMD:C_1206_3216Metric, symbol Device:C_US
- C1: renamed from C31; footprint (none) -> Capacitor_SMD:C_0402_1005Metric
- C10: renamed from C37; footprint (none) -> Capacitor_SMD:C_0201_0603Metric
- C11: renamed from C22; footprint (none) -> Capacitor_SMD:C_0402_1005Metric
- C12: renamed from C38; footprint (none) -> Capacitor_SMD:C_0201_0603Metric
- C13: renamed from C23; footprint (none) -> Capacitor_SMD:C_0402_1005Metric
- C14: renamed from C49; footprint (none) -> Capacitor_SMD:C_0201_0603Metric
- C15: renamed from C52; footprint (none) -> Capacitor_SMD:C_0201_0603Metric
- C18: renamed from C50; footprint (none) -> Capacitor_SMD:C_1206_3216Metric
- C19: renamed from C53; footprint (none) -> Capacitor_SMD:C_1206_3216Metric
- C2: renamed from C27; footprint (none) -> Capacitor_SMD:C_0201_0603Metric
- C22: renamed from C33; footprint (none) -> Capacitor_SMD:C_0201_0603Metric
- C23: renamed from C19; footprint (none) -> Capacitor_SMD:C_0201_0603Metric
- C24: renamed from C34; footprint (none) -> Capacitor_SMD:C_0201_0603Metric
- C25: renamed from C2; footprint (none) -> Capacitor_SMD:C_0402_1005Metric
- C26: renamed from C3; footprint (none) -> Capacitor_SMD:C_0201_0603Metric
- C27: renamed from C4; footprint (none) -> Capacitor_SMD:C_0201_0603Metric
- C28: renamed from C5; footprint (none) -> Capacitor_SMD:C_0201_0603Metric
- C29: renamed from C6; footprint (none) -> Capacitor_SMD:C_0201_0603Metric
- C3: renamed from C28; footprint (none) -> Capacitor_SMD:C_0402_1005Metric
- C30: renamed from C7; footprint (none) -> Capacitor_SMD:C_0201_0603Metric
- C31: renamed from C8; footprint (none) -> Capacitor_SMD:C_0201_0603Metric
- C32: renamed from C9; footprint (none) -> Capacitor_SMD:C_0201_0603Metric
- C33: renamed from C10; footprint (none) -> Capacitor_SMD:C_0201_0603Metric
- C34: renamed from C11; footprint (none) -> Capacitor_SMD:C_0201_0603Metric
- C35: renamed from C12; footprint (none) -> Capacitor_SMD:C_0201_0603Metric
- C36: renamed from C13; footprint (none) -> Capacitor_SMD:C_0201_0603Metric
- C37: renamed from C14; footprint (none) -> Capacitor_SMD:C_0402_1005Metric
- C38: renamed from C1; footprint (none) -> Capacitor_SMD:C_0201_0603Metric
- C39: renamed from C24; footprint (none) -> Capacitor_SMD:C_0201_0603Metric
- C4: renamed from C35; footprint (none) -> Capacitor_SMD:C_0201_0603Metric
- C40: renamed from C32; footprint (none) -> Capacitor_SMD:C_0201_0603Metric
- C41: renamed from C44; footprint (none) -> Capacitor_SMD:C_0201_0603Metric
- C42: renamed from C40; footprint (none) -> Capacitor_SMD:C_0201_0603Metric
- C43: renamed from C15; footprint (none) -> Capacitor_SMD:C_0201_0603Metric
- C44: renamed from C16; footprint (none) -> Capacitor_SMD:C_0201_0603Metric
- C45: renamed from C25; footprint (none) -> Capacitor_SMD:C_0201_0603Metric
- C46: renamed from C26; footprint (none) -> Capacitor_SMD:C_0201_0603Metric
- C47: renamed from C39; footprint (none) -> Capacitor_SMD:C_0201_0603Metric
- C48: renamed from C45; footprint (none) -> Capacitor_SMD:C_0201_0603Metric
- C49: renamed from C46; footprint (none) -> Capacitor_SMD:C_0201_0603Metric
- C5: renamed from C20; footprint (none) -> Capacitor_SMD:C_0201_0603Metric
- C50: renamed from C17; footprint (none) -> Capacitor_SMD:C_0201_0603Metric
- C51: renamed from C29; footprint (none) -> Capacitor_SMD:C_0201_0603Metric
- C52: renamed from C41; footprint (none) -> Capacitor_SMD:C_0201_0603Metric
- C53: renamed from C47; footprint (none) -> Capacitor_SMD:C_0201_0603Metric
- C54: renamed from C18; footprint (none) -> Capacitor_SMD:C_0402_1005Metric
- C55: renamed from C30; footprint (none) -> Capacitor_SMD:C_0402_1005Metric
- C56: renamed from C42; footprint (none) -> Capacitor_SMD:C_0402_1005Metric
- C57: renamed from C48; footprint (none) -> Capacitor_SMD:C_0402_1005Metric
- C6: renamed from C21; footprint (none) -> Capacitor_SMD:C_0201_0603Metric
- C7: renamed from C36; footprint (none) -> Capacitor_SMD:C_0201_0603Metric
- C8: renamed from C43; footprint (none) -> Capacitor_SMD:C_0201_0603Metric
- C9: renamed from C51; footprint (none) -> Capacitor_SMD:C_0201_0603Metric
- FB1: renamed from FB2; value 220 @ 100MHZ -> 220 @ 100 MHz; footprint (none) -> Inductor_SMD:L_0201_0603Metric
- FB2: renamed from FB3; value 220 @ 100MHz -> 220 @ 100 MHz; footprint (none) -> Inductor_SMD:L_0201_0603Metric
- FB3: renamed from FB1; footprint (none) -> Inductor_SMD:L_0201_0603Metric
- FB4, FB5, FB6: footprint (none) -> Inductor_SMD:L_0201_0603Metric
- J1, J2, J3, J4: footprint (none) -> Connector_USB:USB3_A_Molex_48393-001
- P1: footprint (none) -> Connector_USB:USB_C_Plug_JAE_DX07P024AJ1
- R1: footprint (none) -> Resistor_SMD:R_0402_1005Metric
- R10: renamed from R4; footprint (none) -> Resistor_SMD:R_0402_1005Metric
- R11: renamed from R2; footprint (none) -> Resistor_SMD:R_0402_1005Metric
- R12: renamed from R6; footprint (none) -> Resistor_SMD:R_0402_1005Metric
- R13: renamed from R7; footprint (none) -> Resistor_SMD:R_0402_1005Metric
- R14: renamed from R8; footprint (none) -> Resistor_SMD:R_0402_1005Metric
- R15: renamed from R9; footprint (none) -> Resistor_SMD:R_0402_1005Metric
- R16: renamed from R10; footprint (none) -> Resistor_SMD:R_0402_1005Metric
- R17: renamed from R3; footprint (none) -> Resistor_SMD:R_0402_1005Metric
- R18: renamed from R12; footprint (none) -> Resistor_SMD:R_0402_1005Metric
- R19: renamed from R13; footprint (none) -> Resistor_SMD:R_0402_1005Metric
- R2: renamed from R11; footprint (none) -> Resistor_SMD:R_0402_1005Metric
- R20: renamed from R17; footprint (none) -> Resistor_SMD:R_0402_1005Metric
- R3: renamed from R5; footprint (none) -> Resistor_SMD:R_0402_1005Metric
- R4: renamed from R16; footprint (none) -> Resistor_SMD:R_0402_1005Metric
- R5: renamed from R20; footprint (none) -> Resistor_SMD:R_0402_1005Metric
- R6: renamed from R14; footprint (none) -> Resistor_SMD:R_0402_1005Metric
- R7: renamed from R15; footprint (none) -> Resistor_SMD:R_0402_1005Metric
- R8: renamed from R18; footprint (none) -> Resistor_SMD:R_0402_1005Metric
- R9: renamed from R19; footprint (none) -> Resistor_SMD:R_0402_1005Metric
- Y1: footprint (none) -> Crystal:Crystal_SMD_HC49-SD
- renumbered U3 to U1, U4 to U2, U5 to U3, U6 to U4, U2 to U5, U1 to U6
Connections:
- net +3V3: now also R7.2; no longer R7.1
- net DN1_VBUS: now also C16.1, C20.1
- net DN2_VBUS: now also C17.1, C21.1
- net GND: now also U1.7 (EP), U2.7 (EP), U5.7 (EP), C16.2, C17.2, C20.2, C21.2
- net OVERCUR2Z: now also R7.1; no longer R7.2
- no-connect marks 13 -> 10

Commit message: kdsfjsalkf
Parts:
- removed C42, C43, C44, C45, C46, C47, C48, C49, C5, C6: 0.1uF 0201, Capacitor_SMD:C_0201_0603Metric, symbol Device:C_Small
- removed J1, J2, J3, J4: USB3_A, Connector_USB:USB3_A_Molex_48393-001, symbol Connector:USB3_A
- removed P1: USB_C_Plug, Connector_USB:USB_C_Plug_JAE_DX07P024AJ1, symbol Connector:USB_C_Plug
- removed U6: TUSB8041, Package_DFN_QFN:QFN-64-1EP_9x9mm_P0.5mm_EP6x6mm_ThermalVias, symbol Interface_USB:TUSB8041
- added J5, J6, J7, J8: USB_A, symbol Connector:USB_A
- added P2: USB_C_Plug_USB2.0, symbol Connector:USB_C_Plug_USB2.0
- added U7: TUSB4041I, Package_QFP:HTQFP-64-1EP_10x10mm_P0.5mm_EP8x8mm_Mask4.4x4.4mm_ThermalVias, symbol Interface_USB:TUSB4041I
Connections:
- net DN4_VBUS: no longer C15.1
- net GND: now also J5.4 (GND), J6.4 (GND), J7.4 (GND), J8.4 (GND), P2.A1 (GND), P2.A12 (GND), P2.B1 (GND), P2.B12 (GND), U7.65 (VSS)
- net OVERCUR1Z: now also U7.14 (OVERCUR1z)
- net OVERCUR2Z: now also U7.15 (OVERCUR2z)
- net OVERCUR3Z: now also U7.12 (OVERCUR3z)
- net OVERCUR4Z: now also C15.1, U7.11 (OVERCUR4z)
- net PWRCTL_BATEN1: now also U7.4 (PWRCTL1/BATEN1)
- net PWRCTL_BATEN2: now also U7.3 (PWRCTL2/BATEN2)
- net PWRCTL_BATEN3: now also U7.1 (PWRCTL3/BATEN3)
- net PWRCTL_BATEN4: now also U7.64 (PWRCTL4/BATEN4)
- net SHIELD: now also J5.5 (Shield), J6.5 (Shield), J7.5 (Shield), J8.5 (Shield), P2.S1 (SHIELD)
- net USB_DM_UP: now also P2.A7 (D-), U7.22 (USB_DM_UP)
- net USB_DN1.DM: now also J6.3 (D+), U7.34 (USB_DM_DN1)
- net USB_DN1.DP: now also J6.2 (D-), U7.33 (USB_DP_DN1)
- net USB_DN2.DM: now also J5.3 (D+), U7.42 (USB_DM_DN2)
- net USB_DN2.DP: now also J5.2 (D-), U7.41 (USB_DP_DN2)
- net USB_DN3.DM: now also J7.3 (D+), U7.50 (USB_DM_DN3)
- net USB_DN3.DP: now also J7.2 (D-), U7.49 (USB_DP_DN3)
- net USB_DN4.DM: now also J8.3 (D+), U7.57 (USB_DM_DN4)
- net USB_DN4.DP: now also J8.2 (D-), U7.56 (USB_DP_DN4)
- net USB_DP_UP: now also P2.A6 (D+), U7.21 (USB_DP_UP)
- net VBUS: now also P2.A4 (VBUS), P2.A9 (VBUS), P2.B4 (VBUS), P2.B9 (VBUS)
- net VDD: now reaches C30.2, C31.2, C32.2, C33.2, C34.2, C35.2, C36.2, C37.2, FB2.1
- net VDD: now also U7.19 (VDD), U7.25 (VDD), U7.37 (VDD), U7.45 (VDD), U7.53 (VDD), U7.60 (VDD), U7.63 (VDD)
- net at R14.2: now also U7.17 (TEST)
- net at R16.1: now also U7.10 (GANGED/SMBA2/HS_UP)
- net at R10.2, R11.2: now also U7.16 (USB_VBUS)
- net at C41.2, FB6.2: now also J8.1 (VBUS)
- net at R1.1: now also P2.A5 (CC)
- net at C38.2, FB3.2: now also J6.1 (VBUS)
- net at C39.2, FB4.2: now also J5.1 (VBUS)
- net at C13.2, R3.2, Y1.2: now also U7.29 (XO)
- net at R12.1: now also U7.32 (USB_R1)
- net at C11.2, R3.1, Y1.1: now also U7.30 (XI)
- net at R13.2: now also U7.13 (AUTOENz/HS_SUSPEND)
- net VDD33: now reaches C25.2, C26.2, C27.2, C28.2, C29.2, FB1.2
- net VDD33: now also U7.2 (VDD33), U7.20 (VDD33), U7.31 (VDD33), U7.48 (VDD33)
- net at C23.2: now also U7.18 (GRSTz)
- net at R15.2: now also U7.8 (FULLPWRMGMTz/SMBA1)
- net at C40.2, FB5.2: now also J7.1 (VBUS)
- no-connect marks 10 -> 8
Other:
- moved on the sheet: C1, C2, C3, C50, C51, C52, C53, C54, C55, C56, C57, R17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

Commit message: my life is a pahtay
Parts:
- C10, C12, C14, C15, C16, C17, C2, C22, C23, C24, C26, C27, C28, C29, C30, C31, C32, C33, C34, C35, C36, C38, C39, C4, C40, C41, C50, C51, C52, C53, C7, C8, C9: footprint Capacitor_SMD:C_0201_0603Metric -> Capacitor_SMD:C_0402_1005Metric
- J5, J6, J7, J8: footprint (none) -> easyeda2kicad:USB-A-TH_C42622
- P2: footprint (none) -> easyeda2kicad:USB-C-SMD_14P-P0.80_MC-337
Connections:
- net USB_DM_UP renamed USB_DN
- net USB_DN1.DM renamed USB_DN1.DN
- net USB_DN2.DM renamed USB_DN2.DN
- net USB_DN3.DM renamed USB_DN3.DN
- net USB_DN4.DM renamed USB_DN4.DN
- net USB_DP_UP renamed USB_DP
Changed lines of the file:
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@@
 		)
 	)
-	(label "USB_DN1.DM"
+	(label "USB_DN1.DN"
 		(at 406.4 104.14 180)
 		(effects
@@
 		)
 	)
-	(label "USB_DN4.DM"
+	(label "USB_DN4.DN"
 		(at 406.4 142.24 180)
 		(effects
@@
 		)
 	)
-	(label "USB_DN2.DM"
+	(label "USB_DN2.DN"
 		(at 441.96 149.86 0)
 		(effects
@@
 		)
 	)
-	(label "USB_DM_UP"
+	(label "USB_DN"
 		(at 311.15 127 180)
 		(effects
@@
 		)
 	)
-	(label "USB_DN4.DM"
+	(label "USB_DN4.DN"
 		(at 441.96 311.15 0)
 		(effects
@@
 		)
 	)
-	(label "USB_DN3.DM"
+	(label "USB_DN3.DN"
 		(at 406.4 129.54 180)
 		(effects
@@
 		)
 	)
-	(label "USB_DN3.DM"
+	(label "USB_DN3.DN"
 		(at 441.96 219.71 0)
 		(effects
@@
 		)
 	)
-	(label "USB_DN2.DM"
+	(label "USB_DN2.DN"
 		(at 406.4 116.84 180)
 		(effects
@@
 		)
 	)
-	(label "USB_DM_UP"
+	(label "USB_DN"
 		(at 139.7 105.41 0)
 		(effects
@@
 		)
 	)
-	(label "USB_DP_UP"
+	(label "USB_DP"
 		(at 139.7 110.49 0)
 		(effects
@@
 		)
 	)
-	(label "USB_DP_UP"
+	(label "USB_DP"
 		(at 311.15 124.46 180)
 		(effects
@@
 		)
 	)
-	(label "USB_DN1.DM"
+	(label "USB_DN1.DN"
 		(at 441.96 74.93 0)
 		(effects
@@
 			)
 		)
-		(property "Footprint" "Capacitor_SMD:C_0201_0603Metric"
+		(property "Footprint" "Capacitor_SMD:C_0402_1005Metric"
 			(at 350.52 86.36 0)
 			(effects
@@
 			)
 		)
-		(property "Footprint" ""
+		(property "Footprint" "easyeda2kicad:USB-A-TH_C42622"
 			(at 468.63 312.42 0)
 			(effects
@@
 			)
 		)
-		(property "Footprint" "Capacitor_SMD:C_0201_0603Metric"
+		(property "Footprint" "Capacitor_SMD:C_0402_1005Metric"
 			(at 478.4852 95.25 0)
 			(effects
@@
 			)
 		)
-		(property "Footprint" "Capacitor_SMD:C_0201_0603Metric"
+		(property "Footprint" "Capacitor_SMD:C_0402_1005Metric"
 			(at 262.89 226.06 0)
 			(effects
@@
 			)
 		)
-		(property "Footprint" "Capacitor_SMD:C_0201_0603Metric"
+		(property "Footprint" "Capacitor_SMD:C_0402_1005Metric"
 			(at 458.1652 69.85 0)
 			(effects
@@
 			)
 		)
-		(property "Footprint" ""
+		(property "Footprint" "easyeda2kicad:USB-A-TH_C42622"
 			(at 468.63 151.13 0)
 			(effects
@@
 			)
 		)
-		(property "Datasheet" ""
+		(property "Datasheet" "https://www.lcsc.com/datasheet/C528968.pdf?spm=wm.fly.bg.0.pdf___wm.ssy.tc.2.tz&lcsc_vid=QwMKBAAEEVheBVRUFFkKAlQAEVZZBgZfRgcMAgAHFAUxVlNeRFJYUFdXRFRdXzsOAxUeFF5JWBYZEEoKFBINSQcJGk4%3D"
 			(at 293.37 361.95 0)
 			(effects
@@
 			)
 		)
-		(property "Footprint" "Capacitor_SMD:C_0201_0603Metric"
+		(property "Footprint" "Capacitor_SMD:C_0402_1005Metric"
 			(at 355.6 86.36 0)
 			(effects
@@
 			)
 		)
-		(property "Footprint" "Capacitor_SMD:C_0201_0603Metric"
+		(property "Footprint" "Capacitor_SMD:C_0402_1005Metric"
 			(at 215.5952 349.25 0)
 			(effects
@@
 			)
 		)
-		(property "Footprint" "Capacitor_SMD:C_0201_0603Metric"
+		(property "Footprint" "Capacitor_SMD:C_0402_1005Metric"
 			(at 242.57 226.06 0)
 			(effects
@@
 			)
 		)
-		(property "Footprint" ""
+		(property "Footprint" "easyeda2kicad:USB-C-SMD_14P-P0.80_MC-337"
 			(at 121.92 107.95 0)
 			(effects
@@
 			)
 		)
-		(property "Footprint" ""
+		(property "Footprint" "easyeda2kicad:USB-A-TH_C42622"
 			(at 468.63 76.2 0)
 			(effects
@@
 			)
 		)
-		(property "Footprint" "Capacitor_SMD:C_0201_0603Metric"
+		(property "Footprint" "Capacitor_SMD:C_0402_1005Metric"
 			(at 458.1652 144.78 0)
 			(effects
@@
 			)
 		)
-		(property "Footprint" "Capacitor_SMD:C_0201_0603Metric"
+		(property "Footprint" "Capacitor_SMD:C_0402_1005Metric"
 			(at 317.8048 300.99 0)
 			(effects
@@
 			)
 		)
-		(property "Footprint" "Capacitor_SMD:C_0201_0603Metric"
+		(property "Footprint" "Capacitor_SMD:C_0402_1005Metric"
 			(at 330.2 86.36 0)
 			(effects
@@
 			)
 		)
-		(property "Footprint" "Capacitor_SMD:C_0201_0603Metric"
+		(property "Footprint" "Capacitor_SMD:C_0402_1005Metric"
 			(at 335.28 86.36 0)
 			(effects
@@
 			)
 		)
-		(property "Footprint" "Capacitor_SMD:C_0201_0603Metric"
+		(property "Footprint" "Capacitor_SMD:C_0402_1005Metric"
 			(at 340.36 86.36 0)
 			(effects
@@
 			)
 		)
-		(property "Footprint" "Capacitor_SMD:C_0201_0603Metric"
+		(property "Footprint" "Capacitor_SMD:C_0402_1005Metric"
 			(at 317.5 110.7948 0)
 			(effects
@@
 			)
 		)
-		(property "Footprint" "Capacitor_SMD:C_0201_0603Metric"
+		(property "Footprint" "Capacitor_SMD:C_0402_1005Metric"
 			(at 298.45 224.79 0)
 			(effects
@@
 			)
 		)
-		(property "Footprint" "Capacitor_SMD:C_0201_0603Metric"
+		(property "Footprint" "Capacitor_SMD:C_0402_1005Metric"
 			(at 478.4852 170.18 0)
 			(effects
@@
 			)
 		)
-		(property "Footprint" "Capacitor_SMD:C_0201_0603Metric"
+		(property "Footprint" "Capacitor_SMD:C_0402_1005Metric"
 			(at 327.66 86.36 0)
 			(effects
@@
 			)
 		)
-		(property "Footprint" ""
+		(property "Footprint" "easyeda2kicad:USB-A-TH_C42622"
 			(at 468.63 220.98 0)
 			(effects
@@
 			)
 		)
-		(property "Footprint" "Capacitor_SMD:C_0201_0603Metric"
+		(property "Footprint" "Capacitor_SMD:C_0402_1005Metric"
 			(at 345.44 86.36 0)
 			(effects
@@
 			)
 		)
-		(property "Footprint" "Capacitor_SMD:C_0201_0603Metric"
+		(property "Footprint" "Capacitor_SMD:C_0402_1005Metric"
 			(at 458.1652 306.07 0)
 			(effects
@@
 			)
 		)
-		(property "Footprint" "Capacitor_SMD:C_0201_0603Metric"
+		(property "Footprint" "Capacitor_SMD:C_0402_1005Metric"
 			(at 478.4852 331.47 0)
 			(effects
@@
 			)
 		)
-		(property "Footprint" "Capacitor_SMD:C_0201_0603Metric"
+		(property "Footprint" "Capacitor_SMD:C_0402_1005Metric"
 			(at 111.4552 146.05 0)
 			(effects
@@
 			)
 		)
-		(property "Datasheet" ""
+		(property "Datasheet" "https://www.lcsc.com/datasheet/C528968.pdf?spm=wm.fly.bg.0.pdf___wm.ssy.tc.2.tz&lcsc_vid=QwMKBAAEEVheBVRUFFkKAlQAEVZZBgZfRgcMAgAHFAUxVlNeRFJYUFdXRFRdXzsOAxUeFF5JWBYZEEoKFBINSQcJGk4%3D"
 			(at 313.69 297.18 0)
 			(effects
@@
 			)
 		)
-		(property "Datasheet" ""
+		(property "Datasheet" "https://www.lcsc.com/datasheet/C528968.pdf?spm=wm.fly.bg.0.pdf___wm.ssy.tc.2.tz&lcsc_vid=QwMKBAAEEVheBVRUFFkKAlQAEVZZBgZfRgcMAgAHFAUxVlNeRFJYUFdXRFRdXzsOAxUeFF5JWBYZEEoKFBINSQcJGk4%3D"
 			(at 292.1 308.61 0)
 			(effects
@@
 			)
 		)
-		(property "Footprint" "Capacitor_SMD:C_0201_0603Metric"
+		(property "Footprint" "Capacitor_SMD:C_0402_1005Metric"
 			(at 187.96 226.06 0)
 			(effects
@@
 			)
 		)
-		(property "Footprint" "Capacitor_SMD:C_0201_0603Metric"
+		(property "Footprint" "Capacitor_SMD:C_0402_1005Metric"
 			(at 342.9 86.36 0)
 			(effects
@@
 			)
 		)
-		(property "Datasheet" ""
+		(property "Datasheet" "https://www.lcsc.com/datasheet/C528968.pdf?spm=wm.fly.bg.0.pdf___wm.ssy.tc.2.tz&lcsc_vid=QwMKBAAEEVheBVRUFFkKAlQAEVZZBgZfRgcMAgAHFAUxVlNeRFJYUFdXRFRdXzsOAxUeFF5JWBYZEEoKFBINSQcJGk4%3D"
 			(at 313.69 350.52 0)
 			(effects
@@
 			)
 		)
-		(property "Footprint" "Capacitor_SMD:C_0201_0603Metric"
+		(property "Footprint" "Capacitor_SMD:C_0402_1005Metric"
 			(at 215.5952 295.91 0)
 			(effects
@@
 			)
 		)
-		(property "Footprint" "Capacitor_SMD:C_0201_0603Metric"
+		(property "Footprint" "Capacitor_SMD:C_0402_1005Metric"
 			(at 332.74 86.36 0)
 			(effects
@@
 			)
 		)
-		(property "Footprint" "Capacitor_SMD:C_0201_0603Metric"
+		(property "Footprint" "Capacitor_SMD:C_0402_1005Metric"
 			(at 353.06 86.36 0)
 			(effects
@@
 			)
 		)
-		(property "Footprint" "Capacitor_SMD:C_0201_0603Metric"
+		(property "Footprint" "Capacitor_SMD:C_0402_1005Metric"
 			(at 318.77 224.79 0)
 			(effects
@@
 			)
 		)
-		(property "Footprint" "Capacitor_SMD:C_0201_0603Metric"
+		(property "Footprint" "Capacitor_SMD:C_0402_1005Metric"
 			(at 208.28 226.06 0)
 			(effects
@@
 			)
 		)
-		(property "Footprint" "Capacitor_SMD:C_0201_0603Metric"
+		(property "Footprint" "Capacitor_SMD:C_0402_1005Metric"
 			(at 287.9852 312.42 0)
 			(effects
@@
 			)
 		)
-		(property "Footprint" "Capacitor_SMD:C_0201_0603Metric"
+		(property "Footprint" "Capacitor_SMD:C_0402_1005Metric"
 			(at 289.2552 365.76 0)
 			(effects
@@
 			)
 		)
-		(property "Footprint" "Capacitor_SMD:C_0201_0603Metric"
+		(property "Footprint" "Capacitor_SMD:C_0402_1005Metric"
 			(at 478.4852 240.03 0)
 			(effects
@@
 			)
 		)
-		(property "Footprint" "Capacitor_SMD:C_0201_0603Metric"
+		(property "Footprint" "Capacitor_SMD:C_0402_1005Metric"
 			(at 458.1652 214.63 0)
 			(effects
@@
 			)
 		)
-		(property "Footprint" "Capacitor_SMD:C_0201_0603Metric"
+		(property "Footprint" "Capacitor_SMD:C_0402_1005Metric"
 			(at 347.98 86.36 0)
 			(effects
@@
 			)
 		)
-		(property "Footprint" "Capacitor_SMD:C_0201_0603Metric"
+		(property "Footprint" "Capacitor_SMD:C_0402_1005Metric"
 			(at 317.8048 354.33 0)
 			(effects

Commit message: dsklfjsalk
Parts:
- removed Y1: 24MHZ, Crystal:Crystal_SMD_HC49-SD, symbol Device:Crystal
- added Y1: Crystal_GND24, Crystal:Crystal_SMD_3225-4Pin_3.2x2.5mm, symbol Device:Crystal_GND24
- P2: footprint easyeda2kicad:USB-C-SMD_14P-P0.80_MC-337 -> Connector_USB:USB_C_Plug_JAE_DX07P024AJ1
Connections:
- net GND: now also Y1.2, Y1.4
- net at C13.2, R3.2, U7.29 (XO): now also Y1.3
- net at C11.2, R3.1, U7.30 (XI): now also Y1.1

Commit message: dsppfjalk
Connections:
- net SHIELD: no longer C50.1, C51.1, C52.1, C53.1, C54.1, C55.1, C56.1, C57.1, J5.5 (Shield), J6.5 (Shield), J7.5 (Shield), J8.5 (Shield), R17.1, R18.1, R19.1, R20.1
- new net SHIELD1: C50.1, C54.1, J6.5 (Shield), R17.1
- new net SHIELD2: C51.1, C55.1, J5.5 (Shield), R18.1
- new net SHIELD3: C52.1, C56.1, J7.5 (Shield), R19.1
- new net SHIELD4: C53.1, C57.1, J8.5 (Shield), R20.1
Changed lines of the file:
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@@
 		)
 	)
-	(label "SHIELD"
+	(label "SHIELD4"
 		(at 511.81 323.85 180)
 		(effects
@@
 		)
 	)
-	(label "SHIELD"
+	(label "SHIELD2"
 		(at 511.81 162.56 180)
 		(effects
@@
 		)
 	)
-	(label "SHIELD"
+	(label "SHIELD3"
 		(at 511.81 232.41 180)
 		(effects
@@
 		)
 	)
-	(label "SHIELD"
+	(label "SHIELD1"
 		(at 511.81 87.63 180)
 		(effects

Commit message: lkdsnfl
Parts:
- removed C41, C53: 0.1uF, Capacitor_SMD:C_0402_1005Metric, symbol Device:C
- removed C57: 0.001uF, Capacitor_SMD:C_0402_1005Metric, symbol Device:C
- removed FB6: 220 @ 100 MHz, Inductor_SMD:L_0201_0603Metric, symbol Device:FerriteBead
- removed J8: USB_A, easyeda2kicad:USB-A-TH_C42622, symbol Connector:USB_A
- removed R20: 1M, Resistor_SMD:R_0402_1005Metric, symbol Device:R
Connections:
- net OVERCUR4Z: no longer U7.11 (OVERCUR4z)
- net PWRCTL_BATEN4: no longer U7.64 (PWRCTL4/BATEN4)
- net USB_DN4.DN: no longer names the net of U7.57 (USB_DM_DN4)
- net USB_DN4.DP: no longer names the net of U7.56 (USB_DP_DN4)
- no-connect marks 8 -> 12

Commit message: dkslfalk
Parts:
- removed C15: 0.1uF, Capacitor_SMD:C_0402_1005Metric, symbol Device:C
- removed C19: 150uF, Capacitor_SMD:C_1206_3216Metric, symbol Device:C_US
- removed R9: 10K 0402 5%, Resistor_SMD:R_0402_1005Metric, symbol Device:R
Connections:
- net DN4_VBUS: no longer names the net of U4.8 (OUT2)
- net OVERCUR4Z: no longer names the net of U4.6 (~{FAULT2})
- net PWRCTL_BATEN4: no longer names the net of U4.5 (EN2)
- no-connect marks 12 -> 15
