File: USB OverDrive.kicad_pcb (KiCad board)
At the start: 4 copper layers, 40.2 x 69.6 mm, 95 parts, among them J1 USB3_A, J2 USB3_A, J3 USB3_A, J4 USB3_A, P1 USB_C_Plug, U1 5.0V, U2 3.3V, U3 TPS2561, U4 TPS2561, U5 1.1V, U6 TUSB8041, Y1 24MHZ

Commit message: my life is a pahtay
Parts:
- removed C42, C43, C44, C45, C46, C47, C48, C49, C5, C6: 0.1uF 0201, Capacitor_SMD:C_0201_0603Metric
- removed J1, J2, J3, J4: USB3_A, Connector_USB:USB3_A_Molex_48393-001
- removed P1: USB_C_Plug, Connector_USB:USB_C_Plug_JAE_DX07P024AJ1
- removed U6: TUSB8041, Package_DFN_QFN:QFN-64-1EP_9x9mm_P0.5mm_EP6x6mm_ThermalVias
- added J5: USB_A, easyeda2kicad:USB-A-TH_C42622, F.Cu at (120.1, 142.8)
- added J6: USB_A, easyeda2kicad:USB-A-TH_C42622, F.Cu at (120.1, 126.9)
- added J7: USB_A, easyeda2kicad:USB-A-TH_C42622, F.Cu at (120.1, 111.1)
- added J8: USB_A, easyeda2kicad:USB-A-TH_C42622, F.Cu at (120.1, 95.3)
- added P2: USB_C_Plug_USB2.0, Connector_USB:USB_C_Plug_JAE_DX07P024AJ1, F.Cu at (156.1, 93.7)
- added U7: TUSB4041I, Package_QFP:HTQFP-64-1EP_10x10mm_P0.5mm_EP8x8mm_Mask4.4x4.4mm_ThermalVias, F.Cu at (135.7, 96.7)
- C1, C20, C21, C3, C37, FB2, FB3, FB4, R2, R4, R6, R7, U3, Y1: moved to F.Cu
- C10, C12, C14, C15, C22, C23, C24, C29, C30, C31, C32, C33, C34, C35, C36, C38, C39, C4, C40, C41, C50, C51, C52, C53, C7, C9: footprint Capacitor_SMD:C_0201_0603Metric -> Capacitor_SMD:C_0402_1005Metric
- C16, C17, C2, C26, C27, C28, C8: footprint Capacitor_SMD:C_0201_0603Metric -> Capacitor_SMD:C_0402_1005Metric; moved to F.Cu
- moved R9 57.2 mm to (132.9, 128.6)
- moved R5 57.0 mm to (129.9, 130.6)
- moved R1 54.0 mm to (129.9, 122.6)
- moved R20 53.6 mm to (138.7, 130.6)
- moved R19 53.6 mm to (138.7, 128.6)
- moved R18 53.6 mm to (138.7, 126.6)
- moved FB1 51.3 mm to (144.2, 90.3)
- moved C14 49.8 mm to (132.8, 108.8)
- moved U4 45.1 mm to (145.5, 111.9), turned to 0 degrees
- moved FB2 44.1 mm to (144.2, 92.1), turned to 0 degrees
- moved R17 44.0 mm to (138.7, 124.6)
- moved U5 42.9 mm to (145.7, 140.7), turned to 0 degrees
- moved FB5 42.2 mm to (144.2, 97.3)
- moved FB6 42.2 mm to (144.2, 99.1)
- moved C51 42.1 mm to (141.4, 104.9)
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Connections:
- net Net-(C25-Pad2) renamed /VDD33
- net Net-(C30-Pad2) renamed /VDD
- net SHIELD renamed /SHIELD
- C15 pad 1: /DN4_VBUS -> /OVERCUR4Z
Routing:
- net /SHIELD: track 159.7 -> 0.00 mm, vias 2 -> 0
- net VBUS: track 53.7 -> 0.00 mm, vias 2 -> 0
- net /VDD: track 36.2 -> 0.00 mm, vias 1 -> 0
- net /PWRCTL_BATEN2: track 34.8 -> 0.00 mm, vias 1 -> 0
- net /PWRCTL_BATEN1: track 33.5 -> 0.00 mm, vias 1 -> 0
- net +1V1: track 33.0 -> 0.00 mm, vias 2 -> 0
- net /VDD33: track 30.9 -> 0.00 mm, vias 4 -> 0
- net /USB_DN1.SSTXP: track 28.3 -> 0.00 mm
- net /USB_DN1.SSTXM: track 28.3 -> 0.00 mm
- net /OVERCUR2Z: track 23.1 -> 0.00 mm, vias 2 -> 0
- net Net-(U7-XO): track 21.9 -> 0.00 mm, vias 1 -> 0
- net /DN2_VBUS: track 21.3 -> 0.00 mm, vias 2 -> 0
- net /OVERCUR1Z: track 21.3 -> 0.00 mm, vias 2 -> 0
- net Net-(U7-XI): track 20.7 -> 0.00 mm, vias 1 -> 0
- net /DN1_VBUS: track 19.7 -> 0.00 mm, vias 4 -> 0
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- removed copper zone on In1.Cu, net +3V3
- removed copper zone on B.Cu, net GND
- removed copper zone on F.Cu, net GND
- removed copper zone on In2.Cu, net GND
Other:
- board size 40.2 x 69.6 mm -> 5 x 8.2 mm

Commit message: dsklfjsalk
Parts:
- Y1: value 24MHZ -> Crystal_GND24; footprint Crystal:Crystal_SMD_HC49-SD -> Crystal:Crystal_SMD_3225-4Pin_3.2x2.5mm
- moved U7 28.4 mm to (150.8, 72.6)
- moved Y1 11.7 mm to (128.7, 95.6)
- moved J5 0.53 mm to (119.9, 143.3)
- moved J8 0.50 mm to (119.9, 94.8)
- moved J6 0.25 mm to (119.9, 127.1)
- moved J7 0.24 mm to (119.9, 111.0)
Connections:
- Y1 pad 2: Net-(U7-XO) -> GND
Other:
- board size 5 x 8.2 mm -> 47.2 x 64.3 mm
Changed lines of the file:
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@@
 		)
 	)
-	(footprint "Crystal:Crystal_SMD_HC49-SD"
+	(footprint "Crystal:Crystal_SMD_3225-4Pin_3.2x2.5mm"
 		(layer "F.Cu")
-		(at 135.8175 86.345)
-		(descr "SMD Crystal HC-49-SD http://cdn-reichelt.de/documents/datenblatt/B400/xxx-HC49-SMD.pdf, 11.4x4.7mm^2 package")
+		(at 128.65 95.61)
+		(descr "SMD Crystal SERIES SMD3225/4 http://www.txccrystal.com/images/pdf/7m-accuracy.pdf, 3.2x2.5mm^2 package")
 		(tags "SMD SMT crystal")
 		(property "Reference" "Y1"
-			(at 0 -3.55 0)
+			(at 0 -2.45 0)
 			(layer "F.SilkS")
 			(effects
@@
 			)
 		)
-		(property "Value" "24MHZ"
-			(at 0 3.55 0)
+		(property "Value" "Crystal_GND24"
+			(at 0 2.45 0)
 			(layer "F.Fab")
 			(effects
@@
 			)
 		)
-		(property "Datasheet" "https://jlcpcb.com/partdetail/YXC_CrystalOscillators-X49SD24MSD2SC/C2213"
+		(property "Datasheet" ""
 			(at 0 0 0)
 			(unlocked yes)
@@
 			)
 		)
-		(property "Description" "Two pin crystal"
+		(property "Description" "Four pin crystal, GND on pins 2 and 4"
 			(at 0 0 0)
 			(unlocked yes)
@@
 		(attr smd)
 		(fp_line
-			(start -6.7 -2.55)
-			(end -6.7 2.55)
-			(stroke
-				(width 0.12)
-				(type solid)
-			)
-			(layer "F.SilkS")
-		)
-		(fp_line
-			(start -6.7 2.55)
-			(end 5.9 2.55)
+			(start -2 -1.65)
+			(end -2 1.65)
 			(stroke
 				(width 0.12)
@@
 		)
 		(fp_line
-			(start 5.9 -2.55)
-			(end -6.7 -2.55)
+			(start -2 1.65)
+			(end 2 1.65)
 			(stroke
 				(width 0.12)
@@
 		)
 		(fp_line
-			(start -6.8 -2.6)
-			(end -6.8 2.6)
+			(start -2.1 -1.7)
+			(end -2.1 1.7)
 			(stroke
 				(width 0.05)
@@
 		)
 		(fp_line
-			(start -6.8 2.6)
-			(end 6.8 2.6)
+			(start -2.1 1.7)
+			(end 2.1 1.7)
 			(stroke
 				(width 0.05)
@@
 		)
 		(fp_line
-			(start 6.8 -2.6)
-			(end -6.8 -2.6)
+			(start 2.1 -1.7)
+			(end -2.1 -1.7)
 			(stroke
 				(width 0.05)
@@
 		)
 		(fp_line
-			(start 6.8 2.6)
-			(end 6.8 -2.6)
+			(start 2.1 1.7)
+			(end 2.1 -1.7)
 			(stroke
 				(width 0.05)
@@
 		)
 		(fp_line
-			(start -5.7 -2.35)
-			(end -5.7 2.35)
+			(start -1.6 -1.25)
+			(end -1.6 1.25)
 			(stroke
 				(width 0.1)
@@
 		)
 		(fp_line
-			(start -5.7 2.35)
-			(end 5.7 2.35)
+			(start -1.6 0.25)
+			(end -0.6 1.25)
 			(stroke
 				(width 0.1)
@@
 		)
 		(fp_line
-			(start -3.015 -2.115)
-			(end 3.015 -2.115)
+			(start -1.6 1.25)
+			(end 1.6 1.25)
 			(stroke
 				(width 0.1)
@@
 		)
 		(fp_line
-			(start -3.015 2.115)
-			(end 3.015 2.115)
+			(start 1.6 -1.25)
+			(end -1.6 -1.25)
 			(stroke
 				(width 0.1)
@@
 		)
 		(fp_line
-			(start 5.7 -2.35)
-			(end -5.7 -2.35)
-			(stroke
-				(width 0.1)
-				(type solid)
-			)
-			(layer "F.Fab")
-		)
-		(fp_line
-			(start 5.7 2.35)
-			(end 5.7 -2.35)
-			(stroke
-				(width 0.1)
-				(type solid)
-			)
-			(layer "F.Fab")
-		)
-		(fp_arc
-			(start -3.015 2.115)
-			(mid -5.13 0)
-			(end -3.015 -2.115)
-			(stroke
-				(width 0.1)
-				(type solid)
-			)
-			(layer "F.Fab")
-		)
-		(fp_arc
-			(start 3.015 -2.115)
-			(mid 5.13 0)
-			(end 3.015 2.115)
+			(start 1.6 1.25)
+			(end 1.6 -1.25)
 			(stroke
 				(width 0.1)
@@
 			(effects
 				(font
-					(size 1 1)
-					(thickness 0.15)
+					(size 0.7 0.7)
+					(thickness 0.105)
 				)
 			)
 		)
 		(pad "1" smd rect
-			(at -4.25 0)
-			(size 4.5 2)
+			(at -1.1 0.85)
+			(size 1.4 1.2)
 			(layers "F.Cu" "F.Mask" "F.Paste")
 			(net 3 "Net-(U7-XI)")
@@
 		)
 		(pad "2" smd rect
-			(at 4.25 0)
-			(size 4.5 2)
+			(at 1.1 0.85)
+			(size 1.4 1.2)
 			(layers "F.Cu" "F.Mask" "F.Paste")
-			(net 4 "Net-(U7-XO)")
+			(net 1 "GND")
 			(pinfunction "2")
 			(pintype "passive")
 		)
+		(pad "3" smd rect
+			(at 1.1 -0.85)
+			(size 1.4 1.2)
+			(layers "F.Cu" "F.Mask" "F.Paste")
+			(net 4 "Net-(U7-XO)")
+			(pinfunction "3")
+			(pintype "passive")
+		)
+		(pad "4" smd rect
+			(at -1.1 -0.85)
+			(size 1.4 1.2)
+			(layers "F.Cu" "F.Mask" "F.Paste")
+			(net 1 "GND")
+			(pinfunction "4")
+			(pintype "passive")
+		)
 		(embedded_fonts no)
-		(model "${KICAD9_3DMODEL_DIR}/Crystal.3dshapes/Crystal_SMD_HC49-SD.wrl"
+		(model "${KICAD9_3DMODEL_DIR}/Crystal.3dshapes/Crystal_SMD_3225-4Pin_3.2x2.5mm.wrl"
 			(offset
 				(xyz 0 0 0)
@@
 	(footprint "easyeda2kicad:USB-A-TH_C42622"
 		(layer "F.Cu")
-		(at 120.0725 95.315 -90)
+		(at 119.8875 94.8475 -90)
 		(property "Reference" "J8"
 			(at 0 -4.725 90)
@@
 	(footprint "easyeda2kicad:USB-A-TH_C42622"
 		(layer "F.Cu")
-		(at 120.0725 126.945 -90)
+		(at 119.8875 127.119833 -90)
 		(property "Reference" "J6"
 			(at 0 -4.725 90)
@@
 	(footprint "easyeda2kicad:USB-A-TH_C42622"
 		(layer "F.Cu")
-		(at 120.0725 111.13 -90)
+		(at 119.8875 110.982166 -90)
 		(property "Reference" "J7"
 			(at 0 -4.725 90)
@@
 	(footprint "easyeda2kicad:USB-A-TH_C42622"
 		(layer "F.Cu")
-		(at 120.0725 142.76 -90)
+		(at 119.8875 143.2575 -90)
 		(property "Reference" "J5"
 			(at 0 -4.725 90)
@@
 	(footprint "Package_QFP:HTQFP-64-1EP_10x10mm_P0.5mm_EP8x8mm_Mask4.4x4.4mm_ThermalVias"
 		(layer "F.Cu")
-		(at 135.7175 96.695)
+		(at 150.82 72.61)
 		(descr "64-Lead Plastic Thin Quad Flatpack (PT) - 10x10x1 mm Body, 2.00 mm Footprint [HTQFP] thermal pad")
 		(tags "HTQFP-64 Pitch 0.5 ")
@@
 	)
 	(gr_line
+		(start 154.135 86.9)
+		(end 107.2125 86.9)
+		(stroke
+			(width 0.05)
+			(type solid)
+		)
+		(layer "Edge.Cuts")
+	)
+	(gr_line
+		(start 107.2125 86.9)
+		(end 107.13 86.9)
+		(stroke
+			(width 0.05)
+			(type solid)
+		)
+		(layer "Edge.Cuts")
+	)
+	(gr_line
+		(start 106.98 86.9)
+		(end 106.98 151.2)
+		(stroke
+			(width 0.05)
+			(type solid)
+		)
+		(layer "Edge.Cuts")
+	)
+	(gr_line
+		(start 107.13 86.9)
+		(end 106.98 86.9)
+		(stroke
+			(width 0.05)
+			(type solid)
+		)
+		(layer "Edge.Cuts")
+	)
+	(gr_line
+		(start 106.98 151.2)
+		(end 154.1225 151.2)
+		(stroke
+			(width 0.05)
+			(type solid)
+		)
+		(layer "Edge.Cuts")
+	)
+	(gr_line
+		(start 154.1225 151.2)
+		(end 154.1225 97.95)
+		(stroke
+			(width 0.05)
+			(type solid)
+		)
+		(layer "Edge.Cuts")
+	)
+	(gr_line

Commit message: dsppfjalk
Parts:
- moved FB1 54.8 mm to (198.3, 81.4)
- moved FB3 54.8 mm to (198.3, 84.9)
- moved FB4 54.8 mm to (198.3, 86.6)
- moved FB5 54.8 mm to (198.3, 88.4)
- moved FB6 54.8 mm to (198.3, 90.1)
- moved C18 52.5 mm to (193.4, 133.6)
- moved C19 52.5 mm to (193.4, 137.0)
- moved C20 52.5 mm to (193.4, 140.3)
- moved C21 52.5 mm to (193.4, 143.7)
- moved C25 52.5 mm to (188.2, 105.3)
- moved C26 52.5 mm to (188.2, 107.2)
- moved C27 52.5 mm to (188.2, 109.2)
- moved C28 52.5 mm to (188.2, 111.2)
- moved C29 52.5 mm to (188.2, 113.2)
- moved C38 52.5 mm to (191.1, 113.2)
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Connections:
- C50 pad 1: /SHIELD -> /SHIELD1
- C51 pad 1: /SHIELD -> /SHIELD2
- C52 pad 1: /SHIELD -> /SHIELD3
- C53 pad 1: /SHIELD -> /SHIELD4
- C54 pad 1: /SHIELD -> /SHIELD1
- C55 pad 1: /SHIELD -> /SHIELD2
- C56 pad 1: /SHIELD -> /SHIELD3
- C57 pad 1: /SHIELD -> /SHIELD4
- J5 pad 5: /SHIELD -> /SHIELD2
- J6 pad 5: /SHIELD -> /SHIELD1
- J7 pad 5: /SHIELD -> /SHIELD3
- J8 pad 5: /SHIELD -> /SHIELD4
- R17 pad 1: /SHIELD -> /SHIELD1
- R18 pad 1: /SHIELD -> /SHIELD2
- R19 pad 1: /SHIELD -> /SHIELD3
- R20 pad 1: /SHIELD -> /SHIELD4
Routing:
- net VBUS: track 0.00 -> 57.4 mm, vias 0 -> 4
- net /VDD: track 0.00 -> 23.0 mm, vias 0 -> 4
- net +1V1: track 0.00 -> 6.68 mm, vias 0 -> 2
- net /SHIELD: track 0.00 -> 5.92 mm, vias 0 -> 1
- net Net-(P2-CC): track 0.00 -> 4.27 mm
- net +3V3: track 0.00 -> 0.29 mm, vias 0 -> 1
- net +5V: track 0.00 -> 0.24 mm, vias 0 -> 1
- net GND: vias 0 -> 5
- added copper zone on B.Cu, net GND
- added copper zone on F.Cu, net GND
- added copper zone on In1.Cu, net GND
- added copper zone on In2.Cu, net GND
Other:
- board size 47.2 x 64.3 mm -> 47.2 x 65.3 mm

Commit message: lkdsnfl
Parts:
- removed C41, C53: 0.1uF, Capacitor_SMD:C_0402_1005Metric
- removed C57: 0.001uF, Capacitor_SMD:C_0402_1005Metric
- removed FB6: 220 @ 100 MHz, Inductor_SMD:L_0201_0603Metric
- removed J8: USB_A, easyeda2kicad:USB-A-TH_C42622
- removed R20: 1M, Resistor_SMD:R_0402_1005Metric
- moved U1 91.5 mm to (214.6, 123.3)
- moved C34 91.5 mm to (227.6, 111.3)
- moved C35 91.5 mm to (227.6, 113.2)
- moved C36 91.5 mm to (233.8, 112.1)
- moved C4 91.5 mm to (214.0, 120.5)
- moved C10 91.5 mm to (216.8, 120.5)
- moved C22 78.5 mm to (203.1, 134.6)
- moved C30 78.5 mm to (211.5, 135.9)
- moved C32 78.5 mm to (207.8, 142.4)
- moved C33 78.5 mm to (207.8, 144.4)
- moved C37 78.5 mm to (210.6, 137.9)
- moved FB2 78.5 mm to (209.4, 137.4)
- moved U2 78.5 mm to (200.8, 137.4)
- moved U7 78.5 mm to (219.5, 134.1)
- moved C31 78.5 mm to (211.6, 132.4)
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Connections:
- U7 pad 11: /OVERCUR4Z -> unconnected-(U7-OVERCUR4z-Pad11)
- U7 pad 56: /USB_DN4.DP -> unconnected-(U7-USB_DP_DN4-Pad56)
- U7 pad 57: /USB_DN4.DN -> unconnected-(U7-USB_DM_DN4-Pad57)
- U7 pad 64: /PWRCTL_BATEN4 -> unconnected-(U7-PWRCTL4/BATEN4-Pad64)
Routing:
- net VBUS: track 57.4 -> 0.00 mm, vias 4 -> 0
- net /VDD: track 23.0 -> 0.00 mm, vias 4 -> 0
- net +1V1: track 6.68 -> 0.00 mm, vias 2 -> 0
- net /SHIELD: track 5.92 -> 0.00 mm, vias 1 -> 0
- net Net-(P2-CC): track 4.27 -> 0.00 mm
- net +3V3: track 0.29 -> 0.00 mm, vias 1 -> 0
- net +5V: track 0.24 -> 0.00 mm, vias 1 -> 0
- net GND: vias 5 -> 0
- removed copper zone on B.Cu, net GND
- removed copper zone on F.Cu, net GND
- removed copper zone on In1.Cu, net GND
- removed copper zone on In2.Cu, net GND
Other:
- board size 47.2 x 65.3 mm -> 30.1 x 50 mm

Commit message: dkslfalk
Parts:
- removed C15: 0.1uF, Capacitor_SMD:C_0402_1005Metric
- removed C19: 150uF, Capacitor_SMD:C_1206_3216Metric
- removed R9: 10K 0402 5%, Resistor_SMD:R_0402_1005Metric
- moved C36 104.1 mm to (130.2, 121.0), turned to 180 degrees
- moved C34 103.4 mm to (124.3, 110.0), turned to -90 degrees
- moved Y1 102.3 mm to (132.0, 115.8), turned to -90 degrees
- moved C4 99.3 mm to (116.9, 99.6)
- moved FB5 98.6 mm to (111.7, 135.4), turned to -90 degrees
- moved U1 98.5 mm to (118.7, 101.0)
- moved C10 98.5 mm to (120.5, 99.6)
- moved U7 98.4 mm to (122.5, 117.6)
- moved C35 98.0 mm to (129.7, 117.6), turned to 90 degrees
- moved C30 95.3 mm to (116.8, 125.0)
- moved C31 95.1 mm to (116.8, 126.0)
- moved C33 93.7 mm to (120.5, 110.4), turned to 180 degrees
- moved FB4 92.5 mm to (111.8, 119.3), turned to -90 degrees
- moved C32 92.4 mm to (116.8, 127.0)
- moved C37 91.7 mm to (123.3, 110.0), turned to -90 degrees
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Connections:
- U4 pad 5: /PWRCTL_BATEN4 -> unconnected-(U4-EN2-Pad5)
- U4 pad 6: /OVERCUR4Z -> unconnected-(U4-~{FAULT2}-Pad6)
- U4 pad 8: /DN4_VBUS -> unconnected-(U4-OUT2-Pad8)
Routing:
- net VBUS: track 0.00 -> 68.7 mm, vias 0 -> 7
- net /VDD: track 0.00 -> 55.2 mm, vias 0 -> 5
- net /DN1_VBUS: track 0.00 -> 55.2 mm, vias 0 -> 2
- net +5V: track 0.00 -> 47.9 mm, vias 0 -> 3
- net /VDD33: track 0.00 -> 45.7 mm, vias 0 -> 3
- net +3V3: track 0.00 -> 44.7 mm, vias 0 -> 3
- net /DN2_VBUS: track 0.00 -> 43.9 mm, vias 0 -> 2
- net /USB_DN: track 0.00 -> 36.6 mm, vias 0 -> 2
- net /USB_DP: track 0.00 -> 33.7 mm, vias 0 -> 2
- net /USB_DN3.DN: track 0.00 -> 30.2 mm
- net /USB_DN3.DP: track 0.00 -> 30.1 mm
- net /PWRCTL_BATEN2: track 0.00 -> 27.0 mm
- net /USB_DN2.DN: track 0.00 -> 26.3 mm
- net /USB_DN2.DP: track 0.00 -> 26.3 mm
- net /PWRCTL_BATEN1: track 0.00 -> 26.0 mm
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- added copper zone on B.Cu, net GND
- added copper zone on F.Cu, net GND
- added copper zone on In1.Cu, net GND
- added copper zone on In2.Cu, net GND
Other:
- outline, holes or cut-outs redrawn

Commit message: dsaklfh
Parts:
- U5: value 1.1V -> 1.2V
- moved C30 2.00 mm to (116.8, 127.0), turned to 180 degrees
- moved C32 2.00 mm to (116.8, 125.0), turned to 180 degrees
- moved C23 0.98 mm to (130.2, 123.6)
- moved R14 0.98 mm to (130.2, 122.6)
- moved C10 0.96 mm to (120.5, 100.5), turned to -90 degrees
- moved C4 0.94 mm to (116.9, 100.5), turned to -90 degrees
- moved C22 0.93 mm to (124.2, 100.5), turned to -90 degrees
- moved C31 0.08 mm to (116.8, 125.9), turned to 180 degrees
Connections:
- net +1V1 renamed +1V2
Routing:
- net /PWRCTL_BATEN3: track 24.1 -> 20.5 mm
- net Net-(U7-GRSTz): track 2.69 -> 5.01 mm
- net GND: track 7.99 -> 9.05 mm, vias 71 -> 73
- net Net-(U7-TEST): track 2.79 -> 1.98 mm
- net /USB_DN1.DN: track 19.6 -> 20.3 mm

Commit message: fix drc
Routing:
- net /DN3_VBUS: track 13.7 -> 37.4 mm
- net /VDD: track 54.8 -> 64.5 mm, vias 5 -> 9
- net /VDD33: track 45.7 -> 44.9 mm, vias 3 -> 5
- net GND: vias 73 -> 70
Other:
- board size 30.1 x 50 mm -> 30.3 x 50 mm

Commit message: dkasjfkl
Parts:
- added G***: LOGO, LOGO, F.Cu at (121.0, 142.7)
- added G***: LOGO, LOGO, B.Cu at (130.8, 138.8)
- added G***: LOGO, LOGO, B.Cu at (123.2, 118.9)
- added G***: LOGO, LOGO, B.Cu at (115.4, 105.4)
- added G***: LOGO, LOGO, B.Cu at (128.2, 104.4)
- added G***: LOGO, LOGO, F.Cu at (118.6, 106.5)
- added G***: LOGO, LOGO, F.Cu at (116.1, 135.9)
- added G***: LOGO, LOGO, F.Cu at (131.4, 129.9)
- added G***: LOGO, LOGO, F.Cu at (131.5, 141.9)
- added G***: LOGO, LOGO, F.Cu at (131.1, 100.7)
- added G***: LOGO, LOGO, F.Cu at (128.9, 106.6)
- added G***: LOGO, LOGO, F.Cu at (113.6, 123.0)
- added G***: LOGO, LOGO, B.Cu at (117.2, 139.0)
Routing:
- net /SHIELD2: track 18.4 -> 17.7 mm
- net /USB_DP: track 33.7 -> 33.0 mm
- net /USB_DN: track 36.6 -> 35.9 mm, vias 2 -> 0
- net /DN3_VBUS: track 37.4 -> 36.7 mm
- net /USB_DN3.DN: track 30.2 -> 29.6 mm
- net Net-(U7-XI): track 4.64 -> 4.12 mm
- net +1V2: track 2.45 -> 2.44 mm, vias 1 -> 0
