File: USB OverDrive.kicad_pcb (KiCad board)
At the start: 4 copper layers, 30.3 x 50 mm, 89 parts, among them J5 USB_A, J6 USB_A, J7 USB_A, P2 USB_C_Plug_USB2.0, U1 5.0V, U2 3.3V, U3 TPS2561, U4 TPS2561, U5 1.2V, U7 TUSB4041I, Y1 Crystal_GND24

Commit message: skdfjlk
Parts:
- added G***: LOGO, LOGO, B.Cu at (115.4, 113.8)
